Commit message: fix: change joint type

File: src/robot_description/urdf/robot.xacro (robot description, xacro)
@@ -70,6 +70,5 @@
     </gazebo>
     <!-- wheel_right_joint -->
-    <!-- <joint name="wheel_right_joint" type="continuous"> -->
-    <joint name="wheel_right_joint" type="fixed">
+    <joint name="wheel_right_joint" type="continuous">
         <parent link="base_link"/>
         <child link="wheel_right_link"/>
@@ -82,5 +81,5 @@
             <!-- <origin xyz="0 0 0" rpy="0 0 0"/> -->
             <geometry>
-                <cylinder length="0.018" radius="0.033"/>
+                <!-- <cylinder length="0.018" radius="0.033"/> -->
                 <mesh filename="file://$(find robot_description)/meshes/wheel.stl" scale="0.001 0.001 0.001"/>
             </geometry>
@@ -90,5 +89,5 @@
             <!-- <origin xyz="0 0 0" rpy="0 0 0"/> -->
             <geometry>
-                <cylinder length="0.018" radius="0.033"/>
+                <!-- <cylinder length="0.018" radius="0.033"/> -->
                 <mesh filename="file://$(find robot_description)/meshes/wheel.stl" scale="0.001 0.001 0.001"/>
             </geometry>
@@ -104,6 +103,5 @@
     </gazebo>
     <!-- wheel_left_joint -->
-    <!-- <joint name="wheel_left_joint" type="continuous"> -->
-    <joint name="wheel_left_joint" type="fixed">
+    <joint name="wheel_left_joint" type="continuous">
         <parent link="base_link"/>
         <child link="wheel_left_link"/>
@@ -116,5 +114,5 @@
             <!-- <origin xyz="0 0 0" rpy="0 0 0"/> -->
             <geometry>
-                <cylinder length="0.018" radius="0.033"/>
+                <!-- <cylinder length="0.018" radius="0.033"/> -->
                 <mesh filename="file://$(find robot_description)/meshes/wheel.stl" scale="0.001 0.001 0.001"/>
             </geometry>
@@ -124,5 +122,5 @@
             <!-- <origin xyz="0 0 0" rpy="0 0 0"/> -->
             <geometry>
-                <cylinder length="0.018" radius="0.033"/>
+                <!-- <cylinder length="0.018" radius="0.033"/> -->
                 <mesh filename="file://$(find robot_description)/meshes/wheel.stl" scale="0.001 0.001 0.001"/>
             </geometry>
@@ -196,4 +194,5 @@
                     <remapping>~/out:=imu</remapping>
                 </ros>
+                <initial_orientation_as_reference>false</initial_orientation_as_reference>
             </plugin>
         </sensor>
@@ -236,22 +235,22 @@
             <update_rate>50</update_rate>
             <ray>
-            <scan>
-                <horizontal>
-                <samples>360</samples>
-                <resolution>1.000000</resolution>
-                <min_angle>0.000000</min_angle>
-                <max_angle>6.28319</max_angle>
-                </horizontal>
-            </scan>
-            <range>
-                <min>0.080000</min>
-                <max>8.0</max>
-                <resolution>0.001000</resolution>
-            </range>
-            <noise>
-                <type>gaussian</type>
-                <mean>0.0</mean>
-                <stddev>0.0001</stddev>
-            </noise>
+                <scan>
+                    <horizontal>
+                        <samples>360</samples>
+                        <resolution>1.000000</resolution>
+                        <min_angle>0.000000</min_angle>
+                        <max_angle>6.28319</max_angle>
+                    </horizontal>
+                </scan>
+                <range>
+                    <min>0.080000</min>
+                    <max>8.0</max>
+                    <resolution>0.001000</resolution>
+                </range>
+                <noise>
+                    <type>gaussian</type>
+                    <mean>0.0</mean>
+                    <stddev>0.0001</stddev>
+                </noise>
             </ray>
             <plugin name="robot_laserscan" filename="libgazebo_ros_ray_sensor.so">

Commit message: fix: add caster link

File: src/robot_description/urdf/robot.xacro (robot description, xacro)
@@ -84,5 +84,5 @@
                 <mesh filename="file://$(find robot_description)/meshes/wheel.stl" scale="0.001 0.001 0.001"/>
             </geometry>
-            <material name="dark"/>
+            <material name="black"/>
         </visual>
         <collision>
@@ -117,5 +117,5 @@
                 <mesh filename="file://$(find robot_description)/meshes/wheel.stl" scale="0.001 0.001 0.001"/>
             </geometry>
-            <material name="dark"/>
+            <material name="black"/>
         </visual>
         <collision>
@@ -133,4 +133,90 @@
     </link>
     <gazebo reference="left_wheel_link">
+        <material>Gazebo/FlatBlack</material>
+    </gazebo>
+    <!-- caster_front_joint -->
+    <joint name="caster_front_joint" type="fixed">
+        <parent link="base_link"/>
+        <child link="caster_front_link"/>
+        <origin xyz="0.103 0 -0.009" rpy="0 0 0"/>
+        <!-- <axis xyz="0 0 0"/> -->
+    </joint>
+    <!-- caster_front_link -->
+    <link name="caster_front_link">
+        <visual>
+            <!-- <origin xyz="0 0 0" rpy="0 0 0"/> -->
+            <geometry>
+                <mesh filename="file://$(find robot_description)/meshes/caster.stl" scale="0.001 0.001 0.001"/>
+                <!-- <sphere radius="0.005"/> -->
+            </geometry>
+            <material name="LightGrey">
+                <color rgba="0.7 0.7 0.7 1.0"/>
+            </material>
+        </visual>
+        <collision>
+            <!-- <origin xyz="0 0 0" rpy="0 0 0"/> -->
+            <geometry>
+                <mesh filename="file://$(find robot_description)/meshes/caster.stl" scale="0.001 0.001 0.001"/>
+                <!-- <sphere radius="0.005"/> -->
+            </geometry>
+            <surface>
+                <friction>
+                    <ode>
+                    <mu>0.1</mu>
+                    <mu2>0.1</mu2>
+                    </ode>
+                </friction>
+            </surface>
+        </collision>
+        <inertial>
+            <origin xyz="0 0 0" />
+            <mass value="0.005" />
+            <inertia ixx="0.001" ixy="0.0" ixz="0.0" iyy="0.001" iyz="0.0" izz="0.001" />
+        </inertial>
+    </link>
+    <gazebo reference="caster_front_joint">
+        <material>Gazebo/FlatBlack</material>
+    </gazebo>
+    <!-- caster_back_joint -->
+    <joint name="caster_back_joint" type="fixed">
+        <parent link="base_link"/>
+        <child link="caster_back_link"/>
+        <origin xyz="-0.103 0 -0.009" rpy="0 0 0"/>
+        <!-- <axis xyz="0 0 0"/> -->
+    </joint>
+    <!-- caster_back_link -->
+    <link name="caster_back_link">
+        <visual>
+            <!-- <origin xyz="0 0 0" rpy="0 0 0"/> -->
+            <geometry>
+                <mesh filename="file://$(find robot_description)/meshes/caster.stl" scale="0.001 0.001 0.001"/>
+                <!-- <sphere radius="0.005"/> -->
+            </geometry>
+            <material name="LightGrey">
+                <color rgba="0.7 0.7 0.7 1.0"/>
+            </material>
+        </visual>
+        <collision>
+            <!-- <origin xyz="0 0 0" rpy="0 0 0"/> -->
+            <geometry>
+                <mesh filename="file://$(find robot_description)/meshes/caster.stl" scale="0.001 0.001 0.001"/>
+                <!-- <sphere radius="0.005"/> -->
+            </geometry>
+            <surface>
+                <friction>
+                    <ode>
+                    <mu>0.1</mu>
+                    <mu2>0.1</mu2>
+                    </ode>
+                </friction>
+            </surface>
+        </collision>
+        <inertial>
+            <origin xyz="0 0 0" />
+            <mass value="0.005" />
+            <inertia ixx="0.001" ixy="0.0" ixz="0.0" iyy="0.001" iyz="0.0" izz="0.001" />
+        </inertial>
+    </link>
+    <gazebo reference="caster_back_joint">
         <material>Gazebo/FlatBlack</material>
     </gazebo>

Commit message: fix: urdf

File: src/robot_description/urdf/robot.xacro (robot description, xacro)
@@ -99,5 +99,5 @@
         </inertial>
     </link>
-    <gazebo reference="left_wheel_link">
+    <gazebo reference="wheel_right_link">
         <material>Gazebo/FlatBlack</material>
     </gazebo>
@@ -132,5 +132,5 @@
         </inertial>
     </link>
-    <gazebo reference="left_wheel_link">
+    <gazebo reference="wheel_left_link">
         <material>Gazebo/FlatBlack</material>
     </gazebo>
@@ -139,5 +139,5 @@
         <parent link="base_link"/>
         <child link="caster_front_link"/>
-        <origin xyz="0.103 0 -0.009" rpy="0 0 0"/>
+        <origin xyz="0.103 0 -0.0098" rpy="0 0 0"/>
         <!-- <axis xyz="0 0 0"/> -->
     </joint>
@@ -163,6 +163,8 @@
                 <friction>
                     <ode>
-                    <mu>0.1</mu>
-                    <mu2>0.1</mu2>
+                        <mu>1.0</mu>  <!-- 增加摩擦系数 -->
+                        <mu2>1.0</mu2>
+                        <slip1>0.01</slip1>  <!-- 添加滑动参数 -->
+                        <slip2>0.01</slip2>
                     </ode>
                 </friction>
@@ -171,9 +173,9 @@
         <inertial>
             <origin xyz="0 0 0" />
-            <mass value="0.005" />
-            <inertia ixx="0.001" ixy="0.0" ixz="0.0" iyy="0.001" iyz="0.0" izz="0.001" />
-        </inertial>
-    </link>
-    <gazebo reference="caster_front_joint">
+            <mass value="0.05" /> <!-- 从0.005增加到0.05 -->
+            <inertia ixx="0.0001" ixy="0.0" ixz="0.0" iyy="0.0001" iyz="0.0" izz="0.0001" />
+        </inertial>
+    </link>
+    <gazebo reference="caster_front_link">
         <material>Gazebo/FlatBlack</material>
     </gazebo>
@@ -182,5 +184,5 @@
         <parent link="base_link"/>
         <child link="caster_back_link"/>
-        <origin xyz="-0.103 0 -0.009" rpy="0 0 0"/>
+        <origin xyz="-0.103 0 -0.0098" rpy="0 0 0"/>
         <!-- <axis xyz="0 0 0"/> -->
     </joint>
@@ -206,6 +208,8 @@
                 <friction>
                     <ode>
-                    <mu>0.1</mu>
-                    <mu2>0.1</mu2>
+                        <mu>1.0</mu>  <!-- 增加摩擦系数 -->
+                        <mu2>1.0</mu2>
+                        <slip1>0.01</slip1>  <!-- 添加滑动参数 -->
+                        <slip2>0.01</slip2>
                     </ode>
                 </friction>
@@ -214,9 +218,9 @@
         <inertial>
             <origin xyz="0 0 0" />
-            <mass value="0.005" />
-            <inertia ixx="0.001" ixy="0.0" ixz="0.0" iyy="0.001" iyz="0.0" izz="0.001" />
-        </inertial>
-    </link>
-    <gazebo reference="caster_back_joint">
+            <mass value="0.05" /> <!-- 从0.005增加到0.05 -->
+            <inertia ixx="0.0001" ixy="0.0" ixz="0.0" iyy="0.0001" iyz="0.0" izz="0.0001" />
+        </inertial>
+    </link>
+    <gazebo reference="caster_back_link">
         <material>Gazebo/FlatBlack</material>
     </gazebo>

Commit message: fix: add mu1 param for wheel

File: src/robot_description/urdf/robot.xacro (robot description, xacro)
@@ -369,6 +369,6 @@
             <wheel_diameter>0.066</wheel_diameter>
             <robot_base_frame>base_footprint</robot_base_frame>
-            <max_wheel_torque>20</max_wheel_torque>
-            <max_wheel_acceleration>1.0</max_wheel_acceleration>
+            <max_wheel_torque>10</max_wheel_torque>
+            <max_wheel_acceleration>0.5</max_wheel_acceleration>
             <command_topic>cmd_vel</command_topic>
             <odometry_topic>odom</odometry_topic>
@@ -395,3 +395,22 @@
         </plugin>
     </gazebo>
+    <!-- 为轮子添加对称的Gazebo物理属性 -->
+    <gazebo reference="wheel_left_link">
+        <material>Gazebo/FlatBlack</material>
+        <kp>1000000.0</kp>
+        <kd>100.0</kd>
+        <mu1>1.5</mu1>
+        <mu2>1.5</mu2>
+        <minDepth>0.001</minDepth>
+        <maxVel>1.0</maxVel>
+    </gazebo>
+    <gazebo reference="wheel_right_link">
+        <material>Gazebo/FlatBlack</material>
+        <kp>1000000.0</kp>
+        <kd>100.0</kd>
+        <mu1>1.5</mu1>
+        <mu2>1.5</mu2>
+        <minDepth>0.001</minDepth>
+        <maxVel>1.0</maxVel>
+    </gazebo>
 </robot>
